File: design_files/AST1018.sch (EAGLE design)
At the start: 6 parts, among them J1 SM05B, J2 SM05B, J3 BM05B, J4 BM05B, U1 SK6812MINI

Commit message: updated documentation
Parts:
- J1, J2: device tinycircuits:AS-ITM-00340 -> tinycircuits:AS-ITM-00340EDGE
Other:
- note added: "Hand Populated: -"
- note added: "Hand Soldered: -"
- note added: "Horizontal Connectors"
- note added: "Non Populated: J3, J4"
- note added: "Notes: -"
- note added: "Variant: Standard - R"
- note added: "Vertical Connectors"
- note added: "Wireling RGB LED"
- note removed: "NOTES:"
- note removed: "Optional Populate: R1 or R2 or R3 for DIN"
- note removed: "Optional Populate: R4 or R5 or R6 for DOUT"
- note removed: "Serial RGB LED - Double Con."
- note removed: "WS2812b, SK6812, or compatible 3.5mm Serial RGB LED"
- moved on the sheet: C1, J1, J2, J3, J4, U1
